File: astable_multivibrator.sch (KiCad schematic (older format))
At the start: 120 parts, among them Q1 Q_NPN_BCE, Q10 Q_NPN_BCE, Q11 Q_NPN_BCE, Q12 Q_NPN_BCE, Q13 Q_NPN_BCE, Q14 Q_NPN_BCE, Q15 Q_NPN_BCE, Q16 Q_NPN_BCE, Q17 Q_NPN_BCE, Q18 Q_NPN_BCE, Q19 Q_NPN_BCE, Q2 Q_NPN_BCE, Q20 Q_NPN_BCE, Q21 Q_NPN_BCE, Q22 Q_NPN_BCE, Q23 Q_NPN_BCE, Q24 Q_NPN_BCE, Q3 Q_NPN_BCE, Q4 Q_NPN_BCE, Q5 Q_NPN_BCE, Q6 Q_NPN_BCE, Q7 Q_NPN_BCE, Q8 Q_NPN_BCE, Q9 Q_NPN_BCE

Commit message: generated netlist and imported netlist into pcb.
Parts:
- C1, C10, C11, C12, C13, C14, C15, C16, C17, C18, C19, C2, C20, C21, C22, C23, C24, C3, C4, C5, C6, C7, C8, C9: footprint (none) -> Capacitor_SMD:C_0805_2012Metric_Pad1.15x1.40mm_HandSolder
- Q1, Q10, Q11, Q12, Q13, Q14, Q15, Q16, Q17, Q18, Q19, Q2, Q20, Q21, Q22, Q23, Q24, Q3, Q4, Q5, Q6, Q7, Q8, Q9: footprint (none) -> Package_TO_SOT_SMD:SOT-23-6_Handsoldering
- R1, R10, R11, R12, R13, R14, R15, R16, R17, R18, R19, R2, R20, R21, R22, R23, R24, R25, R26, R27, R28, R29, R3, R30, R31, R32, R33, R34, R35, R36, R37, R38, R39, R4, R40, R41, R42, R43, R44, R45, R46, R47, R48, R49, R5, R50, R51, R52, R53, R54, R55, R56, R57, R58, R59, R6, R60, R61, R62, R63, R64, R65, R66, R67, R68, R69, R7, R70, R71, R72, R8, R9: footprint (none) -> Resistor_THT:R_Axial_DIN0204_L3.6mm_D1.6mm_P5.08mm_Horizontal

Commit message: added speaker and usb-mini power plug to schematic.
Parts:
- added D1, D10, D11, D12, D2, D3, D4, D5, D6, D7, D8, D9: DIODE, symbol pspice:DIODE
- added J1: USB_B_Mini, symbol Connector:USB_B_Mini
- added LS1: Speaker_Crystal, symbol Device:Speaker_Crystal
Connections:
- net labels added: Output
- wire segments 276 -> 306
- no-connect marks 0 -> 4

Commit message: Added switches to schematic and labeling to both schematic and PCB
Parts:
- added SW1, SW10, SW11, SW12, SW2, SW3, SW4, SW5, SW6, SW7, SW8, SW9: SW_SPST, symbol Switch:SW_SPST
Connections:
- wire segments 306 -> 317
